File: soundkarte.kicad_sch (KiCad schematic)
At the start: 218 parts, among them J1 JTAG, J2 DB9, J3 Conn_01x05_Pin, J4 Conn_01x06_Pin, J5 Conn_01x08_Pin, J6 Conn_01x02_Pin, J7 Conn_01x02_Pin, J8 Conn_01x02_Pin, Q1 Q_NPN_BEC, Q2 BC807, Q3 BC807, U1 DSP56364, U12 LM78M05_TO252, U13 Opamp_Dual, U14 74HC74, U15 TS274CD, U2 28F640, U3 74LS393, U4 74HC14, U8 LD1086D2M33TR, U9 LD1086D2M33TR, X1 SG-8002JC

Commit message: ba
Parts:
- added C47, C48, C49, C50, C51: 220 35G, Capacitor_SMD:CP_Elec_10x10.5, symbol Device:C_Polarized
- added C52, C53, C54: 22 35G, Capacitor_SMD:CP_Elec_6.3x3, symbol Device:C_Polarized
- added C55, C56, C57: C, Capacitor_SMD:C_0805_2012Metric, symbol Device:C
- added H7: MountingHole_Pad, MountingHole:MountingHole_4mm_Pad, symbol Mechanical:MountingHole_Pad
Connections:
- net +12V: now also U5.16 (VCC), U6.16 (VCC), U7.16 (VCC), C47.1, C48.1, C49.1, C50.1, C51.1, C55.1, C56.1, C57.1
- net GND: now also C47.2, C48.2, C49.2, C50.2, C51.2, C55.2, C56.2, C57.2
- net at Q1.3 (C), TP10.1, U4.4: now also R16.1; no longer R16.2
- net at U1.28 (PINT/NMI): now also R16.2; no longer R16.1
- new net Earth: H7.1

Commit message: reset
Parts:
- added TP87: TestPoint, TestPoint:TestPoint_Pad_D1.0mm, symbol Connector:TestPoint
Connections:
- net RESET: now also TP87.1
Changed lines of the file:
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@@
+	(symbol
+		(lib_id "Connector:TestPoint")
+		(at 63.5 152.4 180)
+		(unit 1)
+		(exclude_from_sim no)
+		(in_bom yes)
+		(on_board yes)
+		(dnp no)
+		(fields_autoplaced yes)
+		(property "Reference" "TP87"
+			(at 66.04 154.4319 0)
+			(effects
+				(font
+					(size 1.27 1.27)
+				)
+				(justify right)
+			)
+		)
+		(property "Value" "TestPoint"
+			(at 66.04 156.9719 0)
+			(effects
+				(font
+					(size 1.27 1.27)
+				)
+				(justify right)
+			)
+		)
+		(property "Footprint" "TestPoint:TestPoint_Pad_D1.0mm"
+			(at 58.42 152.4 0)
+			(effects
+				(font
+					(size 1.27 1.27)
+				)
+				(hide yes)
+			)
+		)
+		(property "Datasheet" "~"
+			(at 58.42 152.4 0)
+			(effects
+				(font
+					(size 1.27 1.27)
+				)
+				(hide yes)
+			)
+		)
+		(property "Description" "test point"
+			(at 63.5 152.4 0)
+			(effects
+				(font
+					(size 1.27 1.27)
+				)
+				(hide yes)
+			)
+		)
+		(pin "1"
+		)
+		(instances
+			(project "soundkarte"
+				(path "/3728182d-43da-45de-af39-f660b583c15d"
+					(reference "TP87")
+					(unit 1)
+				)
+			)
+		)
+	)
 	(symbol
 		(lib_id "Connector:TestPoint")

Commit message: verbindungen
Parts:
- added C58, C59, C60: C, Capacitor_SMD:C_1206_3216Metric, symbol Device:C
- added C61, C62: C, Capacitor_SMD:C_0805_2012Metric, symbol Device:C
- added R39, R40, R41, R42, R43: 10k, Resistor_SMD:R_0805_2012Metric, symbol Device:R
- added TP88, TP89, TP90: TestPoint, TestPoint:TestPoint_Pad_D1.0mm, symbol Connector:TestPoint
- J6: value Conn_01x02_Pin -> LSP R
- J7: value Conn_01x02_Pin -> Sub
- J8: value Conn_01x02_Pin -> LSP L
Connections:
- net +12V: now also C1.1, C11.1, C12.1, C13.1, C14.1, C2.1, C28.1, C29.1, C3.1, L1.2, U12.1 (VI), U8.3 (IN), U9.3 (IN)
- net +3.3V: now also C10.1, C31.1, C33.1, C6.1, R8.1, TP52.1, U1.11 (VCCLQ), U1.37 (VCCLQ), U1.66 (VCCLQ), U1.87 (VCCLQ), U9.2 (OUT), TP88.1
- net +5V: now also TP89.1
- net GND: now also JP1.2 (B), R40.1, R41.1
- net MISO: now reaches TP64.1, TP9.1, U1.5 (FSR), U4.5
- net at U15.1: now also C61.2
- net at TP82.1, U15.2 (-): now also C61.1
- net MOSI: now reaches TP8.1, U1.7 (SCKR), U4.2
- net at TP80.1, U15.6 (-): now also C62.1
- net at U15.7: now also C62.2
- net at TP23.1, U1.40 (WR), U2.55 (WE#): now also R43.1
- net SCLK: now reaches R16.1, TP10.1, U4.4
- net SCLK: no longer Q1.3 (C)
- net ~{SCLK}: now reaches J4.5 (Pin_5), R10.1, R9.2
- net at C34.1, C35.1, C36.1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: now also TP90.1
- net at JP3.1 (A), TP18.1, U1.1 (MODD): now also R41.2
- net ~{MISO}: now reaches C18.1, J4.1 (Pin_1)
- net ~{MISO}: now also R15.1
- net at JP1.1 (A), TP20.1, U1.3 (MODA): now also R39.2
- net at JP2.1 (A), TP19.1, U1.2 (MODB): now also R40.2
- net at R47.2: now also C58.1, C59.1, C60.1
- net Volume: now reaches J4.3 (Pin_3), R36.2, R47.3
- net ~{MOSI}: now reaches J4.4 (Pin_4), R11.2, R12.1
- net at C54.1: now also U7.9 (MUTE)
- net at R16.2, U1.28 (PINT/NMI): now also Q1.3 (C)
- net at TP22.1, U1.41 (RD), U2.54 (OE#): now also R42.1
- new net: R39.1, R42.2, R43.2
Other:
- moved on the sheet: C54

Commit message: testpunkte
Parts:
- removed TP46: TestPoint, TestPoint:TestPoint_Pad_D1.0mm, symbol Connector:TestPoint
- added C63, C64, C65, C66, C67, C68, C69, C70, C73, C74: C, Capacitor_SMD:C_0805_2012Metric, symbol Device:C
- added C71, C72, C75, C76, C77, C78, C79: C, Capacitor_SMD:C_1206_3216Metric, symbol Device:C
- added R44, R45, R46, R49, R51, R52, R53, R54, R55, R56, R57, R58: R, Resistor_SMD:R_0805_2012Metric, symbol Device:R
- added R50: 10k, Resistor_SMD:R_0805_2012Metric, symbol Device:R
- added R59, R60, R61, R62, R63, R64: R, Resistor_SMD:R_0603_1608Metric, symbol Device:R
- added TP100, TP101, TP102, TP103, TP104, TP105, TP106, TP107, TP108, TP109, TP110, TP111, TP112, TP113, TP114, TP115, TP116, TP117, TP118, TP119, TP120, TP121, TP122, TP91, TP92, TP93, TP94, TP95, TP96, TP97, TP98, TP99: TestPoint, TestPoint:TestPoint_Pad_D1.0mm, symbol Connector:TestPoint
Connections:
- net +12V: now also TP92.1
- net +3.3V: now also U1.15 (VCCHQ), U1.35 (VCCHQ), U1.61 (VCCHQ), U1.89 (VCCHQ), C65.2, TP109.1
- net +5V: now also C67.1, C75.2
- net GND: now also C19.2, C20.2, C22.2, C24.2, C25.2, C32.2, C33.2, C52.2, C53.2, C54.2, U1.12 (GNDQ), U1.36 (GNDQ), U1.49 (GNDA), U1.56 (GNDA), U1.64 (GNDA), U1.65 (GNDQ), U1.72 (GNDA), U1.88 (GNDQ), U11.21 (ZERO), U2.2 (CE1), U5.12 (S-GND), U6.12 (S-GND), U7.12 (S-GND), X1.2 (GND), C66.2, C67.2, C70.2, C71.1, C72.1, C75.1, R45.1, R46.1, R49.1, R56.2, TP122.1
- net at U15.12 (+), U15.3 (+), U15.5 (+): now also C70.1
- net at TP75.1, U15.13 (-): now also C69.2, R61.1, R62.1
- net at TP76.1, U15.14: now also C69.1
- net at C61.2, U15.1: now also R64.1
- net at C61.1, TP82.1, U15.2 (-): now also R63.1, R64.2
- net at C62.1, TP80.1, U15.6 (-): now also R59.2, R60.1
- net at C62.2, U15.7: now also R59.1, TP98.1
- net at C59.2: now also R62.2, TP100.1
- net at U14.1 (~{R}), U14.10 (~{S}), U14.13 (~{R})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: now also TP112.1
- net at U14.11 (C): now also TP70.1, U3.11 (Q0)
- net at U14.12 (D), U14.8 (~{Q}): now also TP111.1
- net at U14.9 (Q): now also R58.1
- net at R35.1, R48.3, U13.2 (-): now also R44.2
- net at U3.8 (Q3): now also U3.1 (CP), TP97.1
- net at C46.2, TP81.1, U1.4 (FST)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: now also R57.1
- net at U14.3 (C): now also U3.5 (Q2), TP110.1
- net at R34.1, U13.7: now also R53.2, R54.1, TP103.1
- net at X1.1 (OE): now also R51.2, TP96.1
- net at R19.2, X1.3 (OUT): now also TP93.1
- net at X1.4 (Vcc): now also C66.1, R51.1
- net at R37.2: now also C74.1
- net at TP83.1, U11.13 (VoutR): now also C78.1
- net at U11.14 (AGND1): now also C79.1
- net at C26.1, C38.2, U11.15 (Vcc1)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: now also C71.2
- net at TP85.1, U11.16 (VoutL): now also C76.1, C77.1
- net at TP51.1, U1.6 (SCKT), U10.3 (BCKIN)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: now also C73.2, R58.2
- net at U11.9 (Vcc2R): now also C79.2
- net at R38.1, U1.13 (HCKR), U4.9: now also TP95.1
- net at R38.2: now also C74.2
- net at C19.1, U10.18 (EXTL): now also TP94.1
- net at J3.2 (Pin_2), J5.5 (Pin_5), Q3.2 (E)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: now also TP91.1
- net at U5.14 (IN-): now also TP115.1
- net at U5.15 (IN+): now also TP99.1
- net at U5.8 (SYNC): now also R45.2, TP121.1
- net at U5.9 (MUTE): now also C52.1, TP120.1
- net at R17.2, U1.17 (SDO2/SDI3), U4.13: now also TP108.1
- net at TP48.1, U1.38 (TA): now also R50.1
- net at U13.4 (V-): now also R52.2, TP104.1
- net at U13.8 (V+): now also C63.2, C68.1, R52.1, R53.1
- net at C54.1, U7.9 (MUTE): now also TP116.1
- net at Q1.3 (C), R16.2, U1.28 (PINT/NMI): now also TP107.1
- net at U1.42 (VCCC): now also C64.1
- net at U13.6 (-): now also C63.1, R44.1, TP102.1
- net at U7.8 (SYNC): now also R49.2, TP117.1
- net at C58.2: now also R63.2, TP106.1
- net at C53.1: now also U6.9 (MUTE), TP118.1
- net at TP77.1, U15.10 (+): now also C78.2
- net at C60.2: now also R60.2, TP105.1
- net at U13.3 (+): now also C68.2, R54.2
- net at U15.9 (-): now also R56.1, TP113.1
- net at U6.8 (SYNC): now also R46.2, TP119.1
- net MISO: no longer names the net of TP64.1, TP9.1, U1.5 (FSR), U4.5
- net MOSI: no longer names the net of TP8.1, U1.7 (SCKR), U4.2
- net SCLK: no longer names the net of R16.1, TP10.1, U4.4
- net ~{MISO} renamed ~{FSR}
- net ~{MOSI} renamed ~{SCKR}
- net ~{SCLK} renamed ~{NMI}
- new net: C65.1, R50.2
- new net: C72.2, R55.2, TP114.1
- new net: C76.2, C77.2, R61.2, TP101.1
- no-connect marks 13 -> 18
Other:
- moved on the sheet: C23, C25, C37, C52, C53, C54, C61, C62, J7, J8, TP70, TP75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
